File: pixel_blit.kicad_pcb (KiCad board)
At the start: 2 copper layers, 170.4 x 120.3 mm, 131 parts, among them CN1 PJ-3059-B, J1 Conn_01x03_Pin, SW1 K2-1808SN-A4SW, SW2 DSWB04LHGET, U1 RP2350B_C42415655, U10 DB301V-3.5-3P-GN, U11 DB301V-3.5-3P-GN, U12 DB301V-3.5-3P-GN, U13 DB301V-3.5-3P-GN, U14 DB301V-3.5-3P-GN, U15 DB301V-3.5-3P-GN, U16 DB301V-3.5-3P-GN, U17 DB301V-3.5-3P-GN, U18 DB301V-3.5-3P-GN, U19 DB301V-3.5-3P-GN, U2 W25Q128JVSIQTR, U20 DB301V-3.5-3P-GN, U21 DB301V-3.5-3P-GN, U22 DB301V-3.5-3P-GN, U23 DB301V-3.5-3P-GN, U24 DB301V-3.5-3P-GN, U25 DB301V-3.5-3P-GN, U26 DB301V-3.5-3P-GN, U27 DB301V-3.5-3P-GN, U28 DB301V-3.5-3P-GN, U29 DB301V-3.5-3P-GN, U3 TPS63070RNMR, U30 DB301V-3.5-3P-GN, U31 DB301V-3.5-3P-GN, U32 DB301V-3.5-3P-GN, U33 DB301V-3.5-3P-GN, U34 DB301V-3.5-3P-GN, U35 DB301V-3.5-3P-GN, U36 DB301V-3.5-3P-GN, U37 DB301V-3.5-3P-GN, U38 DB301V-3.5-3P-GN, U39 DB301V-3.5-3P-GN, U40 DB301V-3.5-3P-GN, U41 DSLVDS1048PWR, U42 DSLVDS1047PWR, U43 DBT10-7.62-2P, U44 DBT10-7.62-2P, U45 DBT10-7.62-2P, U46 DBT10-7.62-2P, U47 2.54-1*4, U5 TXS0108EPWR, U6 TXS0108EPWR, U7 TXS0108EPWR, U8 TXS0108EPWR, U9 DB301V-3.5-3P-GN

Commit message: Checkpoint
Parts:
- added H1: MountingHole_Pad, MountingHole:MountingHole_3.2mm_M3_Pad_Via, F.Cu at (223.3, 148.2)
- added H2: MountingHole_Pad, MountingHole:MountingHole_3.2mm_M3_Pad_Via, F.Cu at (223.3, 38.1)
- added H3: MountingHole_Pad, MountingHole:MountingHole_3.2mm_M3_Pad_Via, F.Cu at (59.0, 38.4)
- added H4: MountingHole_Pad, MountingHole:MountingHole_3.2mm_M3_Pad_Via, F.Cu at (58.6, 148.0)
- C16: footprint PCM_JLCPCB:C_0402 -> PCM_JLCPCB:C_0603
- moved U24 173.9 mm to (212.1, 146.2)
- moved U23 164.0 mm to (201.9, 132.9)
- moved U22 154.1 mm to (191.8, 146.2)
- moved U21 143.6 mm to (181.7, 132.9)
- moved U25 137.7 mm to (212.1, 38.3), turned to 180 degrees
- moved U20 136.2 mm to (171.6, 146.2)
- moved U26 128.1 mm to (201.9, 51.5), turned to 180 degrees
- moved SW2 127.7 mm to (60.4, 60.6)
- moved C13 126.8 mm to (252.0, 96.3)
- moved R1 126.8 mm to (248.9, 88.3)
- moved R6 126.8 mm to (251.8, 87.0)
- moved R7 126.8 mm to (248.9, 90.2)
- moved R8 126.8 mm to (248.9, 92.0)
- moved U19 125.2 mm to (161.4, 132.9)
- moved U17 123.9 mm to (141.2, 132.9)
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Connections:
- C16 pad 1: 3V3 -> GND
- C16 pad 2: GND -> +3V3
- C17 pad 1: Net-(C17-Pad1) -> GND
- C17 pad 2: Net-(U1-XIN) -> Net-(C17-Pad2)
- C18 pad 1: Net-(C18-Pad1) -> Net-(U1-XIN)
- C18 pad 2: Net-(C17-Pad1) -> GND
- R6 pad 1: 3V3 -> +3V3
- R9 pad 1: Net-(C18-Pad1) -> Net-(U1-XOUT)
- R9 pad 2: Net-(U1-XOUT) -> Net-(C17-Pad2)
- U1 pad 64: 3V3 -> +3V3
- U35 pad 2: S6_OUT -> S26_OUT
- U41 pad 10: DATA3 -> HS_DATA3
- U41 pad 11: DATA2 -> HS_DATA2
- U41 pad 14: DATA1 -> HS_DATA1
- U41 pad 15: DATA0 -> HS_DATA0
- U42 pad 2: DATA3 -> HS_DATA3
- U42 pad 3: DATA2 -> HS_DATA2
- U42 pad 6: DATA1 -> HS_DATA1
- U42 pad 7: DATA0 -> HS_DATA0
- U5 pad 1: STRING0 -> STRING7
- U5 pad 12: S7_OUT -> S0_OUT
- U5 pad 13: S6_OUT -> S1_OUT
- U5 pad 14: S5_OUT -> S2_OUT
- U5 pad 15: S4_OUT -> S3_OUT
- U5 pad 16: S3_OUT -> S4_OUT
- U5 pad 17: S2_OUT -> S5_OUT
- U5 pad 18: S1_OUT -> S6_OUT
- U5 pad 20: S0_OUT -> S7_OUT
- U5 pad 3: STRING1 -> STRING6
- U5 pad 4: STRING2 -> STRING5
- U5 pad 5: STRING3 -> STRING4
- U5 pad 6: STRING4 -> STRING3
- U5 pad 7: STRING5 -> STRING2
- U5 pad 8: STRING6 -> STRING1
- U5 pad 9: STRING7 -> STRING0
- U6 pad 1: STRING8 -> STRING15
- U6 pad 12: S15_OUT -> S8_OUT
- U6 pad 13: S14_OUT -> S9_OUT
- U6 pad 14: S13_OUT -> S10_OUT
- U6 pad 15: S12_OUT -> S11_OUT
- U6 pad 16: S11_OUT -> S12_OUT
- U6 pad 17: S10_OUT -> S13_OUT
- U6 pad 18: S9_OUT -> S14_OUT
- U6 pad 20: S8_OUT -> S15_OUT
- U6 pad 3: STRING9 -> STRING14
- U6 pad 4: STRING10 -> STRING13
- U6 pad 5: STRING11 -> STRING12
- U6 pad 6: STRING12 -> STRING11
- U6 pad 7: STRING13 -> STRING10
- U6 pad 8: STRING14 -> STRING9
- U6 pad 9: STRING15 -> STRING8
- U7 pad 1: STRING16 -> STRING23
- U7 pad 12: S23_OUT -> S16_OUT
- U7 pad 13: S22_OUT -> S17_OUT
- U7 pad 14: S21_OUT -> S18_OUT
- U7 pad 15: S20_OUT -> S19_OUT
- U7 pad 16: S19_OUT -> S20_OUT
- U7 pad 17: S18_OUT -> S21_OUT
- U7 pad 18: S17_OUT -> S22_OUT
- U7 pad 20: S16_OUT -> S23_OUT
- U7 pad 3: STRING17 -> STRING22
- U7 pad 4: STRING18 -> STRING21
- U7 pad 5: STRING19 -> STRING20
- U7 pad 6: STRING20 -> STRING19
- U7 pad 7: STRING21 -> STRING18
- U7 pad 8: STRING22 -> STRING17
- U7 pad 9: STRING23 -> STRING16
- U8 pad 1: STRING24 -> STRING31
- U8 pad 12: S31_OUT -> S24_OUT
- U8 pad 13: S30_OUT -> S25_OUT
- U8 pad 14: S29_OUT -> S26_OUT
- U8 pad 15: S28_OUT -> S27_OUT
- U8 pad 16: S27_OUT -> S28_OUT
- U8 pad 17: S26_OUT -> S29_OUT
- U8 pad 18: S25_OUT -> S30_OUT
- U8 pad 20: S24_OUT -> S31_OUT
- U8 pad 3: STRING25 -> STRING30
- U8 pad 4: STRING26 -> STRING29
- U8 pad 5: STRING27 -> STRING28
- U8 pad 6: STRING28 -> STRING27
- U8 pad 7: STRING29 -> STRING26
- U8 pad 8: STRING30 -> STRING25
- U8 pad 9: STRING31 -> STRING24
- X1 pad 2: Net-(C17-Pad1) -> GND
- X1 pad 3: Net-(C18-Pad1) -> Net-(C17-Pad2)
- X1 pad 4: Net-(C17-Pad1) -> GND
Routing:
- net S15_OUT: track 0.00 -> 169.3 mm
- net S13_OUT: track 0.00 -> 148.5 mm
- net S14_OUT: track 0.00 -> 147.8 mm
- net S16_OUT: track 0.00 -> 137.0 mm
- net S12_OUT: track 0.00 -> 128.6 mm
- net S11_OUT: track 0.00 -> 125.8 mm
- net S18_OUT: track 0.00 -> 119.7 mm
- net S17_OUT: track 0.00 -> 119.0 mm
- net S9_OUT: track 0.00 -> 109.7 mm
- net S10_OUT: track 0.00 -> 107.6 mm
- net S19_OUT: track 0.00 -> 98.5 mm
- net S20_OUT: track 0.00 -> 95.4 mm
- net S7_OUT: track 0.00 -> 94.2 mm
- net S8_OUT: track 0.00 -> 88.6 mm
- net S21_OUT: track 0.00 -> 80.1 mm
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- added copper zone on B.Cu, net +12V
- added copper zone on F.Cu, net +1V1
- added copper zone on F.Cu, net +3V3
- added copper zone on In2.Cu, net +3V3
- added copper zone on B.Cu, net +5V
- added copper zone on F.Cu, net /VREG_LX
- added copper zone on F.Cu, net GND
- added copper zone on In1.Cu, net GND
- added copper zone on In2.Cu, net GND
Other:
- board size 170.4 x 120.3 mm -> 174.8 x 120.3 mm
- copper layers 2 -> 4

Commit message: Checkpoint
Parts:
- removed C30, C31, C32, C33: 100nF, PCM_JLCPCB:C_0402
- removed JP2: SolderJumper_2_Bridged, Jumper:SolderJumper-2_P1.3mm_Bridged_Pad1.0x1.5mm
- added G***: LOGO, EasyEDA:pixelblitlogo, F.Cu at (120.2, 120.8)
- added R18: 1kΩ, PCM_JLCPCB:R_0402, F.Cu at (138.3, 67.1)
- added R19: 47Ω, PCM_JLCPCB:R_0402, F.Cu at (73.7, 90.8)
- added R24: 47Ω, PCM_JLCPCB:R_0402, F.Cu at (74.8, 90.8)
- added R25: 47Ω, PCM_JLCPCB:R_0402, F.Cu at (75.9, 92.5)
- added R26: 47Ω, PCM_JLCPCB:R_0402, F.Cu at (76.2, 90.8)
- added R27: 47Ω, PCM_JLCPCB:R_0402, F.Cu at (77.2, 92.4)
- added R28: 47Ω, PCM_JLCPCB:R_0402, F.Cu at (77.5, 90.8)
- added R29: 47Ω, PCM_JLCPCB:R_0402, F.Cu at (78.9, 92.0)
- added R30: 47Ω, PCM_JLCPCB:R_0402, F.Cu at (79.2, 91.1)
- added R31: 47Ω, PCM_JLCPCB:R_0402, F.Cu at (89.6, 96.3)
- added R32: 47Ω, PCM_JLCPCB:R_0402, F.Cu at (90.3, 98.2)
- added R33: 47Ω, PCM_JLCPCB:R_0402, F.Cu at (90.9, 96.3)
- added R34: 47Ω, PCM_JLCPCB:R_0402, F.Cu at (91.5, 98.2)
- added R35: 47Ω, PCM_JLCPCB:R_0402, F.Cu at (92.2, 96.3)
- added R36: 47Ω, PCM_JLCPCB:R_0402, F.Cu at (92.9, 98.2)
- added R37: 47Ω, PCM_JLCPCB:R_0402, F.Cu at (93.6, 96.3)
- added R38: 47Ω, PCM_JLCPCB:R_0402, F.Cu at (94.2, 98.1)
- added R39: 47Ω, PCM_JLCPCB:R_0402, F.Cu at (107.2, 81.1)
- added R40: 47Ω, PCM_JLCPCB:R_0402, F.Cu at (109.0, 80.4)
- added R41: 47Ω, PCM_JLCPCB:R_0402, F.Cu at (107.2, 79.8)
- added R42: 47Ω, PCM_JLCPCB:R_0402, F.Cu at (109.0, 79.1)
- added R43: 47Ω, PCM_JLCPCB:R_0402, F.Cu at (107.2, 78.5)
- added R44: 47Ω, PCM_JLCPCB:R_0402, F.Cu at (109.0, 77.8)
- added R45: 47Ω, PCM_JLCPCB:R_0402, F.Cu at (107.2, 77.2)
- added R46: 47Ω, PCM_JLCPCB:R_0402, F.Cu at (107.2, 76.4)
- added R47: 47Ω, PCM_JLCPCB:R_0402, F.Cu at (69.2, 57.4)
- added R48: 47Ω, PCM_JLCPCB:R_0402, F.Cu at (67.4, 58.0)
- added R49: 47Ω, PCM_JLCPCB:R_0402, F.Cu at (69.2, 58.7)
- added R50: 47Ω, PCM_JLCPCB:R_0402, F.Cu at (67.4, 59.3)
- added R51: 47Ω, PCM_JLCPCB:R_0402, F.Cu at (69.2, 60.0)
- added R52: 47Ω, PCM_JLCPCB:R_0402, F.Cu at (67.4, 60.6)
- added R53: 47Ω, PCM_JLCPCB:R_0402, F.Cu at (69.2, 61.3)
- added R54: 47Ω, PCM_JLCPCB:R_0402, F.Cu at (67.4, 61.9)
- added SW3: K2-1808SN-A4SW, EasyEDA:KEY-SMD_4P-L4.2-W3.2-P2.20-LS5.1-TL, F.Cu at (186.3, 111.0)
- added SW4: K2-1808SN-A4SW, EasyEDA:KEY-SMD_4P-L4.2-W3.2-P2.20-LS5.1-TL, F.Cu at (194.6, 111.0)
- added U48: 2.54-1*4, EasyEDA:HDR-TH_4P-P2.54-V-M-1, F.Cu at (159.3, 80.4)
- added U49: 2.54-1*4, EasyEDA:HDR-TH_4P-P2.54-V-M-1, F.Cu at (159.3, 84.2)
- C13: footprint EasyEDA:C0402 -> PCM_JLCPCB:C_0402
- U5, U6, U7, U8: value TXS0108EPWR -> SN74HCT245DBR; footprint EasyEDA:TSSOP-20_L6.5-W4.4-P0.65-LS6.4-BL -> EasyEDA:SSOP-20_L7.2-W5.3-P0.65-LS7.8-BL
- moved R8 189.3 mm to (60.8, 71.1)
- moved R7 188.8 mm to (60.8, 74.1), turned to 180 degrees
- moved C13 186.8 mm to (66.4, 75.4)
- moved R6 179.2 mm to (73.8, 66.4)
- moved R1 111.5 mm to (138.3, 74.1), turned to 90 degrees
- moved SW1 109.2 mm to (134.4, 74.6)
- moved Reset1 108.9 mm to (134.5, 67.7), turned to 180 degrees
- moved C34 95.1 mm to (81.2, 88.8)
- moved C40 94.4 mm to (77.4, 117.0)
- moved C41 94.2 mm to (77.5, 117.9)
- moved C39 89.8 mm to (80.3, 98.0), turned to -90 degrees
- moved C38 89.0 mm to (81.2, 98.0), turned to -90 degrees
- moved C26 83.5 mm to (189.8, 95.9), turned to -90 degrees
- moved C28 83.0 mm to (189.3, 100.1)
- moved C29 82.1 mm to (189.3, 101.3)
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Connections:
- net /VREG_LX renamed VREG_LX
- net Net-(C19-Pad1) renamed 5V_REG
- net Net-(J1-Pin_1) renamed SWCLK
- net Net-(J1-Pin_3) renamed SWDIO
- net Net-(U1-USB_DM) renamed USB_D-
- net Net-(U1-USB_DP) renamed USB_D+
- net Net-(U41-RIN1+) renamed RIN1+
- net Net-(U41-RIN1-) renamed RIN1-
- net Net-(U41-RIN2+) renamed RIN2+
- net Net-(U41-RIN2-) renamed RIN2-
- net Net-(U41-RIN3+) renamed RIN3+
- net Net-(U41-RIN3-) renamed RIN3-
- net Net-(U41-RIN4+) renamed RIN4+
- net Net-(U41-RIN4-) renamed RIN4-
- net Net-(U42-DOUT1+) renamed DOUT1+
- net Net-(U42-DOUT1-) renamed DOUT1-
- net Net-(U42-DOUT2+) renamed DOUT2+
- net Net-(U42-DOUT2-) renamed DOUT2-
- net Net-(U42-DOUT3+) renamed DOUT3+
- net Net-(U42-DOUT3-) renamed DOUT3-
- net Net-(U42-DOUT4+) renamed DOUT4+
- net Net-(U42-DOUT4-) renamed DOUT4-
- net Net-(USB1-DN1) renamed USB_SH_D-
- net Net-(USB1-DP1) renamed USB_SH_D+
- C13 pad 1: GND -> +3V3
- C13 pad 2: Net-(U1-RUN) -> GND
- C18 pad 1: Net-(U1-XIN) -> GND
- C18 pad 2: GND -> Net-(U1-XIN)
- C22 pad 1: Net-(JP2-A) -> +12V
- C23 pad 1: Net-(JP2-A) -> +12V
- C24 pad 1: Net-(JP2-A) -> +12V
- C28 pad 1: Net-(JP1-A) -> +3V3
- C29 pad 1: Net-(JP1-A) -> +3V3
- C34 pad 1: +3V3 -> +5V
- C35 pad 1: +3V3 -> +5V
- C36 pad 1: +3V3 -> +5V
- C37 pad 1: +3V3 -> +5V
- D1 pad 2: Net-(D1-Pad2) -> VBUS
- D2 pad 5: Net-(D1-Pad2) -> VBUS
- JP1 pad 1: Net-(JP1-A) -> +3V3
- PWR_LED1 pad 2: Net-(JP1-A) -> +3V3
- R10 pad 1: Net-(JP2-A) -> +12V
- Reset1 pad 1: Net-(U1-RUN) -> GND
- Reset1 pad 2: unconnected-(Reset1-Pad2) -> GND
- Reset1 pad 3: GND -> Net-(R18-Pad2)
- Reset1 pad 4: GND -> Net-(R18-Pad2)
- SW2 pad 5: 3V3 -> +3V3
- SW2 pad 6: 3V3 -> +3V3
- SW2 pad 7: 3V3 -> +3V3
- SW2 pad 8: 3V3 -> +3V3
- TP2 pad 1: Net-(JP1-A) -> +3V3
- U1 pad 49: STATUS -> unconnected-(U1-GPIO40_ADC0-Pad49)
- U1 pad 52: DATA -> SELECT_BTN
- U1 pad 54: AUDIO_IN -> unconnected-(U1-GPIO43_ADC3-Pad54)
- U1 pad 56: unconnected-(U1-GPIO45_ADC5-Pad56) -> NEXT_BTN
- U1 pad 57: unconnected-(U1-GPIO46_ADC6-Pad57) -> DISP_SDA
- U1 pad 58: unconnected-(U1-GPIO47_ADC7-Pad58) -> DISP_SDL
- U10 pad 2: S1_OUT -> Net-(R24-Pad2)
- U11 pad 2: S2_OUT -> Net-(R25-Pad2)
- U12 pad 2: S3_OUT -> Net-(R26-Pad2)
- U13 pad 2: S4_OUT -> Net-(R27-Pad2)
- U14 pad 2: S5_OUT -> Net-(R28-Pad2)
- U15 pad 2: S6_OUT -> Net-(R29-Pad2)
- U16 pad 2: S7_OUT -> Net-(R30-Pad2)
- U17 pad 2: S8_OUT -> Net-(R31-Pad2)
- U18 pad 2: S9_OUT -> Net-(R32-Pad2)
- U19 pad 2: S10_OUT -> Net-(R33-Pad2)
- U20 pad 2: S11_OUT -> Net-(R34-Pad2)
- U21 pad 2: S12_OUT -> Net-(R35-Pad2)
- U22 pad 2: S13_OUT -> Net-(R36-Pad2)
- U23 pad 2: S14_OUT -> Net-(R37-Pad2)
- U24 pad 2: S15_OUT -> Net-(R38-Pad2)
- U25 pad 2: S16_OUT -> Net-(R39-Pad2)
- U26 pad 2: S17_OUT -> Net-(R40-Pad2)
- U27 pad 2: S18_OUT -> Net-(R41-Pad2)
- U28 pad 2: S19_OUT -> Net-(R42-Pad2)
- U29 pad 2: S20_OUT -> Net-(R43-Pad2)
- U3 pad 12: Net-(JP2-A) -> +12V
- U3 pad 13: Net-(JP2-A) -> +12V
- U30 pad 2: S21_OUT -> Net-(R44-Pad2)
- U31 pad 2: S22_OUT -> Net-(R45-Pad2)
- U32 pad 2: S23_OUT -> Net-(R46-Pad2)
- U33 pad 2: S24_OUT -> Net-(R47-Pad2)
- U34 pad 2: S25_OUT -> Net-(R48-Pad2)
- U35 pad 2: S26_OUT -> Net-(R49-Pad2)
- U36 pad 2: S27_OUT -> Net-(R50-Pad2)
- U37 pad 2: S28_OUT -> Net-(R51-Pad2)
- U38 pad 2: S29_OUT -> Net-(R52-Pad2)
- U39 pad 2: S30_OUT -> Net-(R53-Pad2)
- U4 pad 5: Net-(JP1-A) -> +3V3
- U40 pad 2: S31_OUT -> Net-(R54-Pad2)
- U5 pad 1: STRING7 -> +5V
- U5 pad 10: +5V -> GND
- U5 pad 11: GND -> S8_OUT
- U5 pad 12: S0_OUT -> S9_OUT
- U5 pad 13: S1_OUT -> S10_OUT
- U5 pad 14: S2_OUT -> S11_OUT
- U5 pad 15: S3_OUT -> S12_OUT
- U5 pad 16: S4_OUT -> S13_OUT
- U5 pad 17: S5_OUT -> S14_OUT
- U5 pad 18: S6_OUT -> S15_OUT
- U5 pad 19: +5V -> GND
- U5 pad 2: +3V3 -> STRING15
- U5 pad 20: S7_OUT -> +5V
- U5 pad 3: STRING6 -> STRING14
- U5 pad 4: STRING5 -> STRING13
- U5 pad 5: STRING4 -> STRING12
- U5 pad 6: STRING3 -> STRING11
- U5 pad 7: STRING2 -> STRING10
- U5 pad 8: STRING1 -> STRING9
- U5 pad 9: STRING0 -> STRING8
- U6 pad 1: STRING15 -> +5V
- U6 pad 10: +5V -> GND
- U6 pad 11: GND -> S16_OUT
- U6 pad 12: S8_OUT -> S17_OUT
- U6 pad 13: S9_OUT -> S18_OUT
- U6 pad 14: S10_OUT -> S19_OUT
- U6 pad 15: S11_OUT -> S20_OUT
- U6 pad 16: S12_OUT -> S21_OUT
- U6 pad 17: S13_OUT -> S22_OUT
- U6 pad 18: S14_OUT -> S23_OUT
- U6 pad 19: +5V -> GND
- U6 pad 2: +3V3 -> STRING23
- U6 pad 20: S15_OUT -> +5V
- U6 pad 3: STRING14 -> STRING22
- U6 pad 4: STRING13 -> STRING21
- U6 pad 5: STRING12 -> STRING20
- U6 pad 6: STRING11 -> STRING19
- U6 pad 7: STRING10 -> STRING18
- U6 pad 8: STRING9 -> STRING17
- U6 pad 9: STRING8 -> STRING16
- U7 pad 1: STRING23 -> +5V
- U7 pad 10: +5V -> GND
- U7 pad 11: GND -> S24_OUT
- U7 pad 12: S16_OUT -> S25_OUT
- U7 pad 13: S17_OUT -> S26_OUT
- U7 pad 14: S18_OUT -> S27_OUT
- U7 pad 15: S19_OUT -> S28_OUT
- U7 pad 16: S20_OUT -> S29_OUT
- U7 pad 17: S21_OUT -> S30_OUT
- U7 pad 18: S22_OUT -> S31_OUT
- U7 pad 19: +5V -> GND
- U7 pad 2: +3V3 -> STRING31
- U7 pad 20: S23_OUT -> +5V
- U7 pad 3: STRING22 -> STRING30
- U7 pad 4: STRING21 -> STRING29
- U7 pad 5: STRING20 -> STRING28
- U7 pad 6: STRING19 -> STRING27
- U7 pad 7: STRING18 -> STRING26
- U7 pad 8: STRING17 -> STRING25
- U7 pad 9: STRING16 -> STRING24
- U8 pad 1: STRING31 -> +5V
- U8 pad 10: +5V -> GND
- U8 pad 11: GND -> S0_OUT
- U8 pad 12: S24_OUT -> S1_OUT
- U8 pad 13: S25_OUT -> S2_OUT
- U8 pad 14: S26_OUT -> S3_OUT
- U8 pad 15: S27_OUT -> S4_OUT
- U8 pad 16: S28_OUT -> S5_OUT
- U8 pad 17: S29_OUT -> S6_OUT
- U8 pad 18: S30_OUT -> S7_OUT
- U8 pad 19: +5V -> GND
- U8 pad 2: +3V3 -> STRING7
- U8 pad 20: S31_OUT -> +5V
- U8 pad 3: STRING30 -> STRING6
- U8 pad 4: STRING29 -> STRING5
- U8 pad 5: STRING28 -> STRING4
- U8 pad 6: STRING27 -> STRING3
- U8 pad 7: STRING26 -> STRING2
- U8 pad 8: STRING25 -> STRING1
- U8 pad 9: STRING24 -> STRING0
- U9 pad 2: S0_OUT -> Net-(R19-Pad2)
- USB1 pad 12: unconnected-(USB1-GND-Pad12) -> GND
Routing:
- net NEXT_BTN: track 0.00 -> 206.0 mm, vias 0 -> 2
- net SELECT_BTN: track 0.00 -> 199.2 mm, vias 0 -> 2
- net DISP_SDA: track 0.00 -> 198.3 mm, vias 0 -> 1
- net DISP_SDL: track 0.00 -> 182.3 mm, vias 0 -> 1
- net S15_OUT: track 169.3 -> 3.36 mm
- net Net-(R38-Pad2): track 0.00 -> 152.8 mm
- net S14_OUT: track 147.8 -> 1.55 mm
- net S13_OUT: track 148.5 -> 3.37 mm
- net Net-(R39-Pad2): track 0.00 -> 139.0 mm
- net S16_OUT: track 137.0 -> 1.48 mm
- net Net-(R37-Pad2): track 0.00 -> 134.0 mm
- net Net-(R36-Pad2): track 0.00 -> 133.3 mm
- net S12_OUT: track 128.6 -> 1.56 mm
- net S11_OUT: track 125.8 -> 3.40 mm
- net Net-(R41-Pad2): track 0.00 -> 122.0 mm
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- added copper zone on F.Cu, net +12V
- added copper zone on F.Cu, net +5V
- added copper zone on F.Cu, net 5V_REG
- added copper zone on F.Cu, net L1
- added copper zone on In1.Cu, net L1
- added copper zone on F.Cu, net L2
- added copper zone on In1.Cu, net L2
Other:
- board size 174.8 x 120.3 mm -> 175.5 x 122 mm
- board text added: "+"
- board text added: "-"
- board text added: "12V"
- board text added: "1V1"
- board text added: "3V3"
- board text added: "5V"
- board text added: "6-12VDC"
- board text added: "Board Address"
- board text added: "Boot"
- board text added: "CN1"
- board text added: "CN2"
- board text added: "DATA IN"
- board text added: "DATA OUT"
- board text added: "GND"
- board text added: "I2C OLED"
- board text added: "IR"
- board text added: "Next"
- board text added: "Reset"
- board text added: "SDA"
- board text added: "SDL"
- board text added: "STRING0"
- board text added: "STRING1"
- board text added: "STRING10"
- board text added: "STRING11"
- board text added: "STRING12"
- board text added: "STRING13"
- board text added: "STRING14"
- board text added: "STRING15"
- board text added: "STRING16"
- board text added: "STRING17"
- board text added: "STRING18"
- board text added: "STRING19"
- board text added: "STRING2"
- board text added: "STRING20"
- board text added: "STRING21"
- board text added: "STRING22"
- board text added: "STRING23"
- board text added: "STRING24"
- board text added: "STRING25"
- board text added: "STRING26"
- board text added: "STRING27"
- board text added: "STRING28"
- board text added: "STRING29"
- board text added: "STRING3"
- board text added: "STRING30"
- board text added: "STRING31"
- board text added: "STRING4"
- board text added: "STRING5"
- board text added: "STRING6"
- board text added: "STRING7"
- board text added: "STRING8"
- board text added: "STRING9"
- board text added: "SWC"
- board text added: "SWD"
- board text added: "Select"

Commit message: Close to final, lots of cleanup, added back audio
Parts:
- added C30: 100nF, PCM_JLCPCB:C_0402, F.Cu at (81.5, 82.6)
- added C31: 100nF, PCM_JLCPCB:C_0402, F.Cu at (97.4, 87.6)
- added C32: 100nF, PCM_JLCPCB:C_0402, F.Cu at (99.0, 73.3)
- added C33: 100nF, PCM_JLCPCB:C_0402, F.Cu at (75.9, 61.9)
- added C42: 22nF, PCM_JLCPCB:C_0402, F.Cu at (85.0, 65.3)
- added C43: 1uF, PCM_JLCPCB:C_0402, F.Cu at (110.1, 84.5)
- added C44: 100nF, PCM_JLCPCB:C_0402, F.Cu at (123.5, 87.5)
- added C45: 4.7uF, PCM_JLCPCB:C_0402, F.Cu at (122.1, 87.6)
- added CN2: PJ-3059-B, EasyEDA:AUDIO-TH_XKB_PJ-3059-B, F.Cu at (110.3, 90.8)
- added Card1: TF PUSH, EasyEDA:TF-SMD_TF-PUSH, F.Cu at (105.2, 106.8)
- added D4: SS14, PCM_JLCPCB:D_SMA, F.Cu at (106.5, 88.8)
- added D5: SS14, PCM_JLCPCB:D_SMA, F.Cu at (105.1, 94.2)
- added D6: Red, PCM_JLCPCB:D_0603, F.Cu at (123.2, 94.4)
- added R55: 47kΩ, PCM_JLCPCB:R_0402, F.Cu at (115.3, 77.8)
- added R56: 1kΩ, PCM_JLCPCB:R_0402, F.Cu at (85.0, 64.0)
- added R57: 47kΩ, PCM_JLCPCB:R_0402, F.Cu at (97.8, 105.7)
- added R58: 47kΩ, PCM_JLCPCB:R_0402, F.Cu at (97.6, 111.2)
- added R59: 47kΩ, PCM_JLCPCB:R_0402, F.Cu at (97.8, 106.7)
- added R60: 1kΩ, PCM_JLCPCB:R_0603, F.Cu at (107.3, 84.5)
- added R61: 1kΩ, PCM_JLCPCB:R_0603, F.Cu at (129.8, 95.6)
- added R62: 3362P-1-503LF, EasyEDA:RES-ADJ-TH_3362P, F.Cu at (127.8, 91.0)
- added R65: 1kΩ, PCM_JLCPCB:R_0402, F.Cu at (120.3, 94.4)
- added R66: 1kΩ, PCM_JLCPCB:R_0603, F.Cu at (114.0, 84.5)
- added R67: 470kΩ, PCM_JLCPCB:R_0402, F.Cu at (116.9, 84.4)
- added U50: LMV358IDR, EasyEDA:SOIC-8_L4.9-W3.9-P1.27-LS6.0-BL, F.Cu at (120.7, 90.8)
- R2: value 10kΩ -> 47kΩ
- R3: value 10kΩ -> 100kΩ
- R4: value 10kΩ -> 220kΩ
- R5: value 10kΩ -> 470kΩ
- U5, U6, U7, U8: value SN74HCT245DBR -> SN74LVC8T245PWR; footprint EasyEDA:SSOP-20_L7.2-W5.3-P0.65-LS7.8-BL -> EasyEDA:TSSOP-24_L7.8-W4.4-P0.65-LS6.4-BL
- moved C37 6.16 mm to (65.5, 62.1)
- moved U7 5.12 mm to (69.8, 58.7)
- moved R54 4.61 mm to (63.1, 60.3)
- moved R51 4.61 mm to (64.9, 58.3)
- moved R47 4.61 mm to (64.9, 55.8)
- moved R48 4.61 mm to (63.0, 56.4)
- moved R49 4.61 mm to (64.9, 57.0)
- moved R50 4.61 mm to (63.1, 57.6)
- moved R52 4.61 mm to (63.1, 59.0)
- moved R53 4.61 mm to (64.9, 59.6)
- moved C35 2.47 mm to (97.3, 93.7)
- moved J1 2.18 mm to (98.5, 62.7)
- moved C34 0.95 mm to (81.9, 88.1)
- moved C36 0.78 mm to (105.0, 73.3)
- moved C7 0.37 mm to (82.1, 78.8), turned to -45 degrees
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Connections:
- R2 pad 1: Net-(U1-GPIO36) -> Net-(R2-Pad1)
- R3 pad 1: Net-(U1-GPIO37) -> Net-(R3-Pad1)
- R4 pad 1: Net-(U1-GPIO38) -> Net-(R4-Pad1)
- R5 pad 1: Net-(U1-GPIO39) -> Net-(R5-Pad1)
- SW2 pad 1: Net-(U1-GPIO39) -> Net-(R5-Pad1)
- SW2 pad 2: Net-(U1-GPIO38) -> Net-(R4-Pad1)
- SW2 pad 3: Net-(U1-GPIO37) -> Net-(R3-Pad1)
- SW2 pad 4: Net-(U1-GPIO36) -> Net-(R2-Pad1)
- SW2 pad 5: +3V3 -> Net-(R55-Pad2)
- SW2 pad 6: +3V3 -> Net-(R55-Pad2)
- SW2 pad 7: +3V3 -> Net-(R55-Pad2)
- SW2 pad 8: +3V3 -> Net-(R55-Pad2)
- U1 pad 1: STRING0 -> STRING4
- U1 pad 11: STRING8 -> STRING12
- U1 pad 12: STRING9 -> STRING13
- U1 pad 13: STRING10 -> STRING14
- U1 pad 14: STRING11 -> STRING15
- U1 pad 16: STRING12 -> STRING16
- U1 pad 17: STRING13 -> STRING17
- U1 pad 18: STRING14 -> STRING18
- U1 pad 19: STRING15 -> STRING19
- U1 pad 2: STRING1 -> STRING5
- U1 pad 20: STRING16 -> STRING20
- U1 pad 21: STRING17 -> STRING21
- U1 pad 22: STRING18 -> STRING22
- U1 pad 23: STRING19 -> STRING23
- U1 pad 25: STRING20 -> STRING24
- U1 pad 26: STRING21 -> STRING25
- U1 pad 27: STRING22 -> STRING26
- U1 pad 28: STRING23 -> STRING27
- U1 pad 3: STRING2 -> STRING6
- U1 pad 36: STRING24 -> STRING28
- U1 pad 37: STRING25 -> STRING29
- U1 pad 38: STRING26 -> STRING30
- U1 pad 39: STRING27 -> STRING31
- U1 pad 4: STRING3 -> STRING7
- U1 pad 40: STRING28 -> HS_DATA3
- U1 pad 42: STRING29 -> HS_DATA2
- U1 pad 43: STRING30 -> HS_DATA1
- U1 pad 44: STRING31 -> HS_DATA0
- U1 pad 45: Net-(U1-GPIO36) -> SD_MISO
- U1 pad 46: Net-(U1-GPIO37) -> SD_CS#
- U1 pad 47: Net-(U1-GPIO38) -> SD_SCK
- U1 pad 48: Net-(U1-GPIO39) -> SD_MOSI
- U1 pad 49: unconnected-(U1-GPIO40_ADC0-Pad49) -> Net-(U1-GPIO40_ADC0)
- U1 pad 52: SELECT_BTN -> AUDIO_IN
- U1 pad 54: unconnected-(U1-GPIO43_ADC3-Pad54) -> SELECT_BTN
- U1 pad 6: STRING4 -> STRING8
- U1 pad 7: STRING5 -> STRING9
- U1 pad 77: HS_DATA0 -> STRING0
- U1 pad 78: HS_DATA1 -> STRING1
- U1 pad 79: HS_DATA3 -> STRING2
- U1 pad 8: STRING6 -> STRING10
- U1 pad 80: HS_DATA2 -> STRING3
- U1 pad 9: STRING7 -> STRING11
- U5 pad 1: +5V -> +3V3
- U5 pad 10: GND -> STRING8
- U5 pad 11: S8_OUT -> GND
- U5 pad 12: S9_OUT -> GND
- U5 pad 13: S10_OUT -> GND
- U5 pad 14: S11_OUT -> S8_OUT
- U5 pad 15: S12_OUT -> S9_OUT
- U5 pad 16: S13_OUT -> S10_OUT
- U5 pad 17: S14_OUT -> S11_OUT
- U5 pad 18: S15_OUT -> S12_OUT
- U5 pad 19: GND -> S13_OUT
- U5 pad 2: STRING15 -> +3V3
- U5 pad 20: +5V -> S14_OUT
- U5 pad 3: STRING14 -> STRING15
- U5 pad 4: STRING13 -> STRING14
- U5 pad 5: STRING12 -> STRING13
- U5 pad 6: STRING11 -> STRING12
- U5 pad 7: STRING10 -> STRING11
- U5 pad 8: STRING9 -> STRING10
- U5 pad 9: STRING8 -> STRING9
- U6 pad 1: +5V -> +3V3
- U6 pad 10: GND -> STRING16
- U6 pad 11: S16_OUT -> GND
- U6 pad 12: S17_OUT -> GND
- U6 pad 13: S18_OUT -> GND
- U6 pad 14: S19_OUT -> S16_OUT
- U6 pad 15: S20_OUT -> S17_OUT
- U6 pad 16: S21_OUT -> S18_OUT
- U6 pad 17: S22_OUT -> S19_OUT
- U6 pad 18: S23_OUT -> S20_OUT
- U6 pad 19: GND -> S21_OUT
- U6 pad 2: STRING23 -> +3V3
- U6 pad 20: +5V -> S22_OUT
- U6 pad 3: STRING22 -> STRING23
- U6 pad 4: STRING21 -> STRING22
- U6 pad 5: STRING20 -> STRING21
- U6 pad 6: STRING19 -> STRING20
- U6 pad 7: STRING18 -> STRING19
- U6 pad 8: STRING17 -> STRING18
- U6 pad 9: STRING16 -> STRING17
- U7 pad 1: +5V -> +3V3
- U7 pad 10: GND -> STRING24
- U7 pad 11: S24_OUT -> GND
- U7 pad 12: S25_OUT -> GND
- U7 pad 13: S26_OUT -> GND
- U7 pad 14: S27_OUT -> S24_OUT
- U7 pad 15: S28_OUT -> S25_OUT
- U7 pad 16: S29_OUT -> S26_OUT
- U7 pad 17: S30_OUT -> S27_OUT
- U7 pad 18: S31_OUT -> S28_OUT
- U7 pad 19: GND -> S29_OUT
- U7 pad 2: STRING31 -> +3V3
- U7 pad 20: +5V -> S30_OUT
- U7 pad 3: STRING30 -> STRING31
- U7 pad 4: STRING29 -> STRING30
- U7 pad 5: STRING28 -> STRING29
- U7 pad 6: STRING27 -> STRING28
- U7 pad 7: STRING26 -> STRING27
- U7 pad 8: STRING25 -> STRING26
- U7 pad 9: STRING24 -> STRING25
- U8 pad 1: +5V -> +3V3
- U8 pad 10: GND -> STRING0
- U8 pad 11: S0_OUT -> GND
- U8 pad 12: S1_OUT -> GND
- U8 pad 13: S2_OUT -> GND
- U8 pad 14: S3_OUT -> S0_OUT
- U8 pad 15: S4_OUT -> S1_OUT
- U8 pad 16: S5_OUT -> S2_OUT
- U8 pad 17: S6_OUT -> S3_OUT
- U8 pad 18: S7_OUT -> S4_OUT
- U8 pad 19: GND -> S5_OUT
- U8 pad 2: STRING7 -> +3V3
- U8 pad 20: +5V -> S6_OUT
- U8 pad 3: STRING6 -> STRING7
- U8 pad 4: STRING5 -> STRING6
- U8 pad 5: STRING4 -> STRING5
- U8 pad 6: STRING3 -> STRING4
- U8 pad 7: STRING2 -> STRING3
- U8 pad 8: STRING1 -> STRING2
- U8 pad 9: STRING0 -> STRING1
Routing:
- net AUDIO_IN: track 0.00 -> 141.7 mm
- net HS_DATA3: track 52.9 -> 169.7 mm
- net HS_DATA2: track 51.2 -> 158.9 mm
- net HS_DATA1: track 63.4 -> 158.3 mm
- net HS_DATA0: track 65.8 -> 158.6 mm
- net SD_MOSI: track 0.00 -> 72.1 mm, vias 0 -> 2
- net SD_MISO: track 0.00 -> 70.3 mm, vias 0 -> 2
- net SD_SCK: track 0.00 -> 66.3 mm, vias 0 -> 2
- net SD_CS#: track 0.00 -> 63.6 mm, vias 0 -> 2
- net Net-(U1-GPIO36): track 62.6 -> 0.00 mm, vias 1 -> 0
- net Net-(U1-GPIO39): track 62.4 -> 0.00 mm, vias 1 -> 0
- net Net-(U1-GPIO38): track 62.0 -> 0.00 mm, vias 1 -> 0
- net Net-(U1-GPIO37): track 62.0 -> 0.00 mm, vias 1 -> 0
- net IR_IN: track 82.4 -> 132.1 mm, vias 2 -> 0
- net Net-(R55-Pad2): track 0.00 -> 43.4 mm, vias 0 -> 3
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- added copper zone on B.Cu, net GND
Other:
- board text added: "Audio In"
- board text added: "Audio Level"
