File: output.kicad_sch (KiCad schematic)
At the start: 44 parts, among them U10 DB301V-3.5-3P-GN, U11 DB301V-3.5-3P-GN, U12 DB301V-3.5-3P-GN, U13 DB301V-3.5-3P-GN, U14 DB301V-3.5-3P-GN, U15 DB301V-3.5-3P-GN, U16 DB301V-3.5-3P-GN, U17 DB301V-3.5-3P-GN, U18 DB301V-3.5-3P-GN, U19 DB301V-3.5-3P-GN, U20 DB301V-3.5-3P-GN, U21 DB301V-3.5-3P-GN, U22 DB301V-3.5-3P-GN, U23 DB301V-3.5-3P-GN, U24 DB301V-3.5-3P-GN, U25 DB301V-3.5-3P-GN, U26 DB301V-3.5-3P-GN, U27 DB301V-3.5-3P-GN, U28 DB301V-3.5-3P-GN, U29 DB301V-3.5-3P-GN, U30 DB301V-3.5-3P-GN, U31 DB301V-3.5-3P-GN, U32 DB301V-3.5-3P-GN, U33 DB301V-3.5-3P-GN, U34 DB301V-3.5-3P-GN, U35 DB301V-3.5-3P-GN, U36 DB301V-3.5-3P-GN, U37 DB301V-3.5-3P-GN, U38 DB301V-3.5-3P-GN, U39 DB301V-3.5-3P-GN, U40 DB301V-3.5-3P-GN, U5 TXS0108EPWR, U6 TXS0108EPWR, U7 TXS0108EPWR, U8 TXS0108EPWR, U9 DB301V-3.5-3P-GN

Commit message: Checkpoint
Connections:
- net S0_OUT: now also U5.12 (B8); no longer U5.20 (B1)
- net S10_OUT: now also U6.14 (B6); no longer U6.17 (B3)
- net S11_OUT: now also U6.15 (B5); no longer U6.16 (B4)
- net S12_OUT: now also U6.16 (B4); no longer U6.15 (B5)
- net S13_OUT: now also U6.17 (B3); no longer U6.14 (B6)
- net S14_OUT: now also U6.18 (B2); no longer U6.13 (B7)
- net S15_OUT: now also U6.20 (B1); no longer U6.12 (B8)
- net S16_OUT: now also U7.12 (B8); no longer U7.20 (B1)
- net S17_OUT: now also U7.13 (B7); no longer U7.18 (B2)
- net S18_OUT: now also U7.14 (B6); no longer U7.17 (B3)
- net S19_OUT: now also U7.15 (B5); no longer U7.16 (B4)
- net S1_OUT: now also U5.13 (B7); no longer U5.18 (B2)
- net S20_OUT: now also U7.16 (B4); no longer U7.15 (B5)
- net S21_OUT: now also U7.17 (B3); no longer U7.14 (B6)
- net S22_OUT: now also U7.18 (B2); no longer U7.13 (B7)
- net S23_OUT: now also U7.20 (B1); no longer U7.12 (B8)
- net S24_OUT: now also U8.12 (B8); no longer U8.20 (B1)
- net S25_OUT: now also U8.13 (B7); no longer U8.18 (B2)
- net S26_OUT: now also U35.2, U8.14 (B6); no longer U8.17 (B3)
- net S27_OUT: now also U8.15 (B5); no longer U8.16 (B4)
- net S28_OUT: now also U8.16 (B4); no longer U8.15 (B5)
- net S29_OUT: now also U8.17 (B3); no longer U8.14 (B6)
- net S2_OUT: now also U5.14 (B6); no longer U5.17 (B3)
- net S30_OUT: now also U8.18 (B2); no longer U8.13 (B7)
- net S31_OUT: now also U8.20 (B1); no longer U8.12 (B8)
- net S3_OUT: now also U5.15 (B5); no longer U5.16 (B4)
- net S4_OUT: now also U5.16 (B4); no longer U5.15 (B5)
- net S5_OUT: now also U5.17 (B3); no longer U5.14 (B6)
- net S6_OUT: now also U5.18 (B2); no longer U35.2, U5.13 (B7)
- net S7_OUT: now also U5.20 (B1); no longer U5.12 (B8)
- net S8_OUT: now also U6.12 (B8); no longer U6.20 (B1)
- net S9_OUT: now also U6.13 (B7); no longer U6.18 (B2)
- net STRING0: now also U5.9 (A8); no longer U5.1 (A1)
- net STRING1: now also U5.8 (A7); no longer U5.3 (A2)
- net STRING10: now also U6.7 (A6); no longer U6.4 (A3)
- net STRING11: now also U6.6 (A5); no longer U6.5 (A4)
- net STRING12: now also U6.5 (A4); no longer U6.6 (A5)
- net STRING13: now also U6.4 (A3); no longer U6.7 (A6)
- net STRING14: now also U6.3 (A2); no longer U6.8 (A7)
- net STRING15: now also U6.1 (A1); no longer U6.9 (A8)
- net STRING16: now also U7.9 (A8); no longer U7.1 (A1)
- net STRING17: now also U7.8 (A7); no longer U7.3 (A2)
- net STRING18: now also U7.7 (A6); no longer U7.4 (A3)
- net STRING19: now also U7.6 (A5); no longer U7.5 (A4)
- net STRING2: now also U5.7 (A6); no longer U5.4 (A3)
- net STRING20: now also U7.5 (A4); no longer U7.6 (A5)
- net STRING21: now also U7.4 (A3); no longer U7.7 (A6)
- net STRING22: now also U7.3 (A2); no longer U7.8 (A7)
- net STRING23: now also U7.1 (A1); no longer U7.9 (A8)
- net STRING24: now also U8.9 (A8); no longer U8.1 (A1)
- net STRING25: now also U8.8 (A7); no longer U8.3 (A2)
- net STRING26: now also U8.7 (A6); no longer U8.4 (A3)
- net STRING27: now also U8.6 (A5); no longer U8.5 (A4)
- net STRING28: now also U8.5 (A4); no longer U8.6 (A5)
- net STRING29: now also U8.4 (A3); no longer U8.7 (A6)
- net STRING3: now also U5.6 (A5); no longer U5.5 (A4)
- net STRING30: now also U8.3 (A2); no longer U8.8 (A7)
- net STRING31: now also U8.1 (A1); no longer U8.9 (A8)
- net STRING4: now also U5.5 (A4); no longer U5.6 (A5)
- net STRING5: now also U5.4 (A3); no longer U5.7 (A6)
- net STRING6: now also U5.3 (A2); no longer U5.8 (A7)
- net STRING7: now also U5.1 (A1); no longer U5.9 (A8)
- net STRING8: now also U6.9 (A8); no longer U6.1 (A1)
- net STRING9: now also U6.8 (A7); no longer U6.3 (A2)

Commit message: Checkpoint
Parts:
- removed U5, U6, U7, U8: TXS0108EPWR, EasyEDA:TSSOP-20_L6.5-W4.4-P0.65-LS6.4-BL, symbol EasyEDA:TXS0108EPWR
- added R19, R24, R25, R26, R27, R28, R29, R30, R31, R32, R33, R34, R35, R36, R37, R38, R39, R40, R41, R42, R43, R44, R45, R46, R47, R48, R49, R50, R51, R52, R53, R54: 47Ω, PCM_JLCPCB:R_0402, symbol PCM_JLCPCB-Resistors:0402,47Ω
- added U5, U6, U7, U8: SN74LVC8T245PWR, EasyEDA:TSSOP-24_L7.8-W4.4-P0.65-LS6.4-BL, symbol EasyEDA:SN74LVC8T245PWR
Connections:
- net +3V3: now also C30.1, C31.1, C32.1, C33.1, U5.1 (VCCA), U5.2 (DIR), U6.1 (VCCA), U6.2 (DIR), U7.1 (VCCA), U7.2 (DIR), U8.1 (VCCA), U8.2 (DIR); no longer C34.1, C35.1, C36.1, C37.1
- net +5V: now also C34.1, C35.1, C36.1, C37.1, U5.23 (VCCB), U5.24 (VCCB), U6.23 (VCCB), U6.24 (VCCB), U7.23 (VCCB), U7.24 (VCCB), U8.23 (VCCB), U8.24 (VCCB); no longer C30.1, C31.1, C32.1, C33.1
- net GND: now also U5.11 (GND), U5.12 (GND), U5.13 (GND), U5.22 (~{OE}), U6.11 (GND), U6.12 (GND), U6.13 (GND), U6.22 (~{OE}), U7.11 (GND), U7.12 (GND), U7.13 (GND), U7.22 (~{OE}), U8.11 (GND), U8.12 (GND), U8.13 (GND), U8.22 (~{OE})
- net S0_OUT: now also R19.1, U8.14 (B8); no longer U9.2
- net S10_OUT: now also R33.1, U5.16 (B6); no longer U19.2
- net S11_OUT: now also R34.1, U5.17 (B5); no longer U20.2
- net S12_OUT: now also R35.1, U5.18 (B4); no longer U21.2
- net S13_OUT: now also R36.1, U5.19 (B3); no longer U22.2
- net S14_OUT: now also R37.1, U5.20 (B2); no longer U23.2
- net S15_OUT: now also R38.1, U5.21 (B1); no longer U24.2
- net S16_OUT: now also R39.1, U6.14 (B8); no longer U25.2
- net S17_OUT: now also R40.1, U6.15 (B7); no longer U26.2
- net S18_OUT: now also R41.1, U6.16 (B6); no longer U27.2
- net S19_OUT: now also R42.1, U6.17 (B5); no longer U28.2
- net S1_OUT: now also R24.1, U8.15 (B7); no longer U10.2
- net S20_OUT: now also R43.1, U6.18 (B4); no longer U29.2
- net S21_OUT: now also R44.1, U6.19 (B3); no longer U30.2
- net S22_OUT: now also R45.1, U6.20 (B2); no longer U31.2
- net S23_OUT: now also R46.1, U6.21 (B1); no longer U32.2
- net S24_OUT: now also R47.1, U7.14 (B8); no longer U33.2
- net S25_OUT: now also R48.1, U7.15 (B7); no longer U34.2
- net S26_OUT: now also R49.1, U7.16 (B6); no longer U35.2
- net S27_OUT: now also R50.1, U7.17 (B5); no longer U36.2
- net S28_OUT: now also R51.1, U7.18 (B4); no longer U37.2
- net S29_OUT: now also R52.1, U7.19 (B3); no longer U38.2
- net S2_OUT: now also R25.1, U8.16 (B6); no longer U11.2
- net S30_OUT: now also R53.1, U7.20 (B2); no longer U39.2
- net S31_OUT: now also R54.1, U7.21 (B1); no longer U40.2
- net S3_OUT: now also R26.1, U8.17 (B5); no longer U12.2
- net S4_OUT: now also R27.1, U8.18 (B4); no longer U13.2
- net S5_OUT: now also R28.1, U8.19 (B3); no longer U14.2
- net S6_OUT: now also R29.1, U8.20 (B2); no longer U15.2
- net S7_OUT: now also R30.1, U8.21 (B1); no longer U16.2
- net S8_OUT: now also R31.1, U5.14 (B8); no longer U17.2
- net S9_OUT: now also R32.1, U5.15 (B7); no longer U18.2
- net STRING0: now also U8.10 (A8)
- net STRING1: now also U8.9 (A7)
- net STRING10: now also U5.8 (A6)
- net STRING11: now also U5.7 (A5)
- net STRING12: now also U5.6 (A4)
- net STRING13: now also U5.5 (A3)
- net STRING14: now also U5.4 (A2)
- net STRING15: now also U5.3 (A1)
- net STRING16: now also U6.10 (A8)
- net STRING17: now also U6.9 (A7)
- net STRING18: now also U6.8 (A6)
- net STRING19: now also U6.7 (A5)
- net STRING2: now also U8.8 (A6)
- net STRING20: now also U6.6 (A4)
- net STRING21: now also U6.5 (A3)
- net STRING22: now also U6.4 (A2)
- net STRING23: now also U6.3 (A1)
- net STRING24: now also U7.10 (A8)
- net STRING25: now also U7.9 (A7)
- net STRING26: now also U7.8 (A6)
- net STRING27: now also U7.7 (A5)
- net STRING28: now also U7.6 (A4)
- net STRING29: now also U7.5 (A3)
- net STRING3: now also U8.7 (A5)
- net STRING30: now also U7.4 (A2)
- net STRING31: now also U7.3 (A1)
- net STRING4: now also U8.6 (A4)
- net STRING5: now also U8.5 (A3)
- net STRING6: now also U8.4 (A2)
- net STRING7: now also U8.3 (A1)
- net STRING8: now also U5.10 (A8)
- net STRING9: now also U5.9 (A7)
- new net: R40.2, U26.2
- new net: R29.2, U15.2
- new net: R53.2, U39.2
- new net: R44.2, U30.2
- new net: R30.2, U16.2
- new net: R52.2, U38.2
- new net: R38.2, U24.2
- new net: R27.2, U13.2
- new net: R36.2, U22.2
- new net: R33.2, U19.2
- new net: R51.2, U37.2
- new net: R54.2, U40.2
- new net: R45.2, U31.2
- new net: R26.2, U12.2
- new net: R49.2, U35.2
- new net: R46.2, U32.2
- new net: R50.2, U36.2
- new net: R19.2, U9.2
- new net: R37.2, U23.2
- new net: R25.2, U11.2
- new net: R42.2, U28.2
- new net: R31.2, U17.2
- new net: R34.2, U20.2
- new net: R32.2, U18.2
- new net: R47.2, U33.2
- new net: R48.2, U34.2
- new net: R39.2, U25.2
- new net: R43.2, U29.2
- new net: R41.2, U27.2
- new net: R28.2, U14.2
- new net: R24.2, U10.2
- new net: R35.2, U21.2
Other:
- note added: "Buffers/Level Shifters"
- note added: "Connectors"
- note added: "Series resistors go near the buffers, not the connection"
- note removed: "Level Shifters"
- moved on the sheet: U10, U11, U12, U13, U14, U15, U16, U17, U18, U19, U20, U21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

Commit message: Library shuffle and Fabrication Toolkit micro adjustments
Parts:
- C30, C31, C32, C33, C34, C35, C36, C37: footprint PCM_JLCPCB:C_0402 -> PixelBlit:C_0402; symbol PCM_JLCPCB-Capacitors:0402,100nF -> PixelBlit:0402,100nF
- R19, R24, R25, R26, R27, R28, R29, R30, R31, R32, R33, R34, R35, R36, R37, R38, R39, R40, R41, R42, R43, R44, R45, R46, R47, R48, R49, R50, R51, R52, R53, R54: footprint PCM_JLCPCB:R_0402 -> PixelBlit:R_0402; symbol PCM_JLCPCB-Resistors:0402,47Ω -> PixelBlit:0402,47Ω
- U10, U11, U12, U13, U14, U15, U16, U17, U18, U19, U20, U21, U22, U23, U24, U25, U26, U27, U28, U29, U30, U31, U32, U33, U34, U35, U36, U37, U38, U39, U40, U9: footprint EasyEDA:CONN-TH_DB301V-3.5-3P-GN -> PixelBlit:CONN-TH_DB301V-3.5-3P-GN; symbol EasyEDA:DB301V-3.5-3P-GN -> PixelBlit:DB301V-3.5-3P-GN
- U5, U6, U7, U8: footprint EasyEDA:TSSOP-24_L7.8-W4.4-P0.65-LS6.4-BL -> PixelBlit:TSSOP-24_L7.8-W4.4-P0.65-LS6.4-BL; symbol EasyEDA:SN74LVC8T245PWR -> PixelBlit:SN74LVC8T245PWR

Commit message: Working on errata
Parts:
- added F10, F11, F12, F13, F14, F15, F16, F17, F18, F19, F20, F21, F22, F23, F24, F25, F26, F27, F28, F29, F30, F31, F32, F33, F34, F35, F36, F37, F38, F39, F8, F9: 1812L400/16GR, EasyEDA:F1812, symbol EasyEDA:1812L400_16GR
- renumbered U14 to J10, U15 to J11, U16 to J12, U17 to J13, U18 to J14, U19 to J15, U20 to J16, U21 to J17, U22 to J18, U23 to J19, U24 to J20, U25 to J21, U26 to J22, U27 to J23, U28 to J24, U29 to J25, U30 to J26, U31 to J27, U32 to J28, U33 to J29, U34 to J30, U35 to J31, U36 to J32, U37 to J33, U38 to J34, U39 to J35, U40 to J36, U9 to J5, U10 to J6, U11 to J7, U12 to J8, U13 to J9
Connections:
- removed net +12V: J10.1, J11.1, J12.1, J13.1, J14.1, J15.1, J16.1, J17.1, J18.1, J19.1, J20.1, J21.1, J22.1, J23.1, J24.1, J25.1, J26.1, J27.1, J28.1, J29.1, J30.1, J31.1, J32.1, J33.1, J34.1, J35.1, J36.1, J5.1, J6.1, J7.1, J8.1, J9.1
- new net: F25.2, J22.1
- new net: F23.2, J20.1
- new net: F15.2, J12.1
- new net: F30.2, J27.1
- new net: F12.2, J9.1
- new net: F21.2, J18.1
- new net: F27.2, J24.1
- new net: F18.2, J15.1
- new net: F36.2, J33.1
- new net: F39.2, J36.1
- new net: F35.2, J32.1
- new net: F14.2, J11.1
- new net: F11.2, J8.1
- new net: F10.2, J7.1
- new net: F19.2, J16.1
- new net: F34.2, J31.1
- new net: F31.2, J28.1
- new net: F37.2, J34.1
- new net: F8.2, J5.1
- new net: F26.2, J23.1
- new net: F16.2, J13.1
- new net: F17.2, J14.1
- new net: F22.2, J19.1
- new net: F24.2, J21.1
- new net: F28.2, J25.1
- new net: F38.2, J35.1
- new net: F33.2, J30.1
- new net: F13.2, J10.1
- new net: F32.2, J29.1
- new net: F9.2, J6.1
- new net: F29.2, J26.1
- new net: F20.2, J17.1
- new net +12V_Z1: F11.1, F13.1, F15.1, F17.1, F19.1, F21.1, F23.1, F9.1
- new net +12V_Z2: F10.1, F12.1, F14.1, F16.1, F18.1, F20.1, F22.1, F8.1
- new net +12V_Z3: F25.1, F27.1, F29.1, F31.1, F33.1, F35.1, F37.1, F39.1
- new net +12V_Z4: F24.1, F26.1, F28.1, F30.1, F32.1, F34.1, F36.1, F38.1
Other:
- moved on the sheet: R31, R32, R33, R34, R35, R36, R37, R38, R47, R48, R49, R50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
