File: Power.kicad_sch (KiCad schematic)
At the start: 35 parts, among them U3 TPS63070RNMR, U43 DBT10-7.62-2P, U44 DBT10-7.62-2P, U45 DBT10-7.62-2P, U46 DBT10-7.62-2P, U47 2.54-1*4

Commit message: Checkpoint
Parts:
- removed JP2: SolderJumper_2_Bridged, Jumper:SolderJumper-2_P1.3mm_Bridged_Pad1.0x1.5mm, symbol Jumper:SolderJumper_2_Bridged
- JP1: footprint Jumper:SolderJumper-2_P1.3mm_Bridged_Pad1.0x1.5mm -> (none)
Connections:
- net +12V: now also C22.1, C23.1, C24.1, R10.1, U3.12 (Vin), U3.13 (Vin)
- net +3V3: now also C28.1, C29.1, JP1.1 (A), PWR_LED1.2, TP2.1, U4.5 (VOUT)
- net 5V_REG: now reaches C19.1, C20.1, C21.1, D3.2, R11.1, R12.2, TP3.1, U3.7 (Vout), U3.8 (Vout)
Other:
- note removed: "This is an input jumper to disable 12V supply."

Commit message: Library shuffle and Fabrication Toolkit micro adjustments
Parts:
- C19, C24: footprint PCM_JLCPCB:C_0603 -> PixelBlit:C_0603; symbol PCM_JLCPCB-Capacitors:0603,10uF,(2) -> PixelBlit:0603,10uF,(2)
- C20: footprint PCM_JLCPCB:C_0805 -> PixelBlit:C_0805; symbol PCM_JLCPCB-Capacitors:0805,10uF,(2) -> PixelBlit:0805,10uF,(2)
- C21: footprint PCM_JLCPCB:C_0805 -> PixelBlit:C_0805; symbol PCM_JLCPCB-Capacitors:0805,47uF -> PixelBlit:0805,47uF
- C22, C23: footprint PCM_JLCPCB:C_0805 -> PixelBlit:C_0805; symbol PCM_JLCPCB-Capacitors:0805,22uF -> PixelBlit:0805,22uF
- C25: footprint PCM_JLCPCB:C_0402 -> PixelBlit:C_0402; symbol PCM_JLCPCB-Capacitors:0402,100nF -> PixelBlit:0402,100nF
- C26, C28: footprint PCM_JLCPCB:C_0603 -> PixelBlit:C_0603; symbol PCM_JLCPCB-Capacitors:0603,10uF -> PixelBlit:0603,10uF
- C27, C29: footprint PCM_JLCPCB:C_0603 -> PixelBlit:C_0603; symbol PCM_JLCPCB-Capacitors:0603,100nF -> PixelBlit:0603,100nF
- D3: footprint PCM_JLCPCB:D_SOD-123 -> PixelBlit:D_SOD-123; symbol PCM_JLCPCB-Diodes:Schottky,B5819W -> PixelBlit:Schottky,B5819W
- JP1: symbol Jumper:SolderJumper_2_Bridged -> PixelBlit:SolderJumper_2_Bridged
- L2: footprint EasyEDA:L0805 -> PixelBlit:L0805; symbol EasyEDA:MLI2012F-1R5KT -> PixelBlit:MLI2012F-1R5KT
- PWR_LED1, PWR_LED2, PWR_LED3: footprint PCM_JLCPCB:D_0603 -> PixelBlit:D_0603; symbol PCM_JLCPCB-Diodes:LED,0603,Red -> PixelBlit:LED,0603,Red
- R10: footprint PCM_JLCPCB:R_0603 -> PixelBlit:R_0603; symbol PCM_JLCPCB-Resistors:0603,10kΩ -> PixelBlit:0603,10kΩ
- R11, R13: footprint PCM_JLCPCB:R_0603 -> PixelBlit:R_0603; symbol PCM_JLCPCB-Resistors:0603,100kΩ -> PixelBlit:0603,100kΩ
- R12: footprint EasyEDA:R0402 -> PixelBlit:R0402; symbol EasyEDA:0402WGF5603TCE -> PixelBlit:0402WGF5603TCE
- R14, R16, R17: footprint PCM_JLCPCB:R_0402 -> PixelBlit:R_0402; symbol PCM_JLCPCB-Resistors:0402,1kΩ -> PixelBlit:0402,1kΩ
- R15: footprint PCM_JLCPCB:R_0402 -> PixelBlit:R_0402; symbol PCM_JLCPCB-Resistors:0402,100kΩ -> PixelBlit:0402,100kΩ
- TP2, TP3: footprint TestPoint:TestPoint_Pad_1.0x1.0mm -> PixelBlit:TestPoint_Pad_1.0x1.0mm; symbol Connector:TestPoint -> PixelBlit:TestPoint
- U3: footprint EasyEDA:VQFN-HR-15_L3.0-W2.5-P0.50-BL_TPS63070RNMR -> PixelBlit:VQFN-HR-15_L3.0-W2.5-P0.50-BL_TPS63070RNMR; symbol EasyEDA:TPS63070RNMR -> PixelBlit:TPS63070RNMR
- U4: footprint EasyEDA:SOT-23-5_L3.0-W1.7-P0.95-LS2.8-BR -> PixelBlit:SOT-23-5_L3.0-W1.7-P0.95-LS2.8-BR; symbol EasyEDA:ME6217C33M5G -> PixelBlit:ME6217C33M5G
- U43, U44, U45, U46: footprint EasyEDA:CONN-TH_2P-P7.62_DBT10-7.62-2P -> PixelBlit:CONN-TH_2P-P7.62_DBT10-7.62-2P; symbol EasyEDA:DBT10-7.62-2P -> PixelBlit:DBT10-7.62-2P
- U47: footprint EasyEDA:HDR-TH_4P-P2.54-V-M-1 -> PixelBlit:HDR-TH_4P-P2.54-V-M-1; symbol EasyEDA:2.54-1*4 -> PixelBlit:2.54-1*4

Commit message: Working on errata
Parts:
- removed L2: MLI2012F-1R5KT, PixelBlit:L0805, symbol PixelBlit:MLI2012F-1R5KT
- removed R16, R17: 1kΩ, PixelBlit:R_0402, symbol PixelBlit:0402,1kΩ
- removed U43, U44, U45, U46: DBT10-7.62-2P, PixelBlit:CONN-TH_2P-P7.62_DBT10-7.62-2P, symbol PixelBlit:DBT10-7.62-2P
- added D10: BZT52C15V, EasyEDA:SOD-123_L2.7-W1.6-LS3.7-RD-1, symbol EasyEDA:BZT52C15V
- added D4, D5, D6, D7: SS34, PCM_JLCPCB:D_SMA, symbol PCM_JLCPCB-Diodes:Schottky,SS34
- added F1, F2, F3, F4, F5, F6, F7: 3557-2, EasyEDA:FUSE-TH_4P-L19.8-W6.7_3557-2, symbol EasyEDA:3557-2
- added J1, J2, J3, J4: DBT50G-9.5-2P, EasyEDA:CONN-TH_2P-P9.50_DBT50G-9.5-2P, symbol EasyEDA:DBT50G-9.5-2P
- added L2: FXL0420-1R5-M, EasyEDA:IND-SMD_L4.4-W4.2, symbol EasyEDA:FXL0420-1R5-M
- added R16: 2.2kΩ, PCM_JLCPCB:R_0603, symbol PCM_JLCPCB-Resistors:0603,2.2kΩ
- added R3: 8.2kΩ, PCM_JLCPCB:R_0603, symbol PCM_JLCPCB-Resistors:0603,8.2kΩ
- renumbered U47 to J38
Connections:
- net GND: now also D10.2 (A), J1.2, J2.2, J3.2, J4.2, R16.2, R3.1
- net L1: now also L2.2
- net L2: now also L2.1
- net at PWR_LED2.1: now also R16.1
- net at PWR_LED3.1: now also R3.2
- net +12V renamed +12V_SYS
- net +12V_SYS: now also D10.1 (K), D4.1, D5.1, D6.1, D7.1
- new net +12V_Z1: D4.2, F1.1, F1.2, F5.1, F5.2
- new net +12V_Z2: D5.2, F2.1, F2.2, F5.3, F5.4, F6.1, F6.2
- new net +12V_Z3: D6.2, F3.1, F3.2, F6.3, F6.4, F7.1, F7.2
- new net +12V_Z4: D7.2, F4.1, F4.2, F7.3, F7.4
- new net J1_IN: F1.3, F1.4, J1.1
- new net J2_IN: F2.3, F2.4, J2.1
- new net J3_IN: F3.3, F3.4, J3.1
- new net J4_IN: F4.3, F4.4, J4.1
Other:
- moved on the sheet: PWR_LED3

Commit message: Fixes for second production run
Parts:
- removed F1, F2, F3, F4, F5, F6, F7: 3557-2, EasyEDA:FUSE-TH_4P-L19.8-W6.7_3557-2, symbol EasyEDA:3557-2
- added F1, F2, F3, F4, F5, F6, F7: XF-507P, JLCImport:XF-507P, symbol JLCImport:XF-507P
Connections:
- net +12V_Z1: now also F1.1, F1.2, F5.1, F5.2
- net +12V_Z2: now also F2.1, F2.2, F5.3, F5.4, F6.1, F6.2
- net +12V_Z3: now also F3.1, F3.2, F6.3, F6.4, F7.1, F7.2
- net +12V_Z4: now also F4.1, F4.2, F7.3, F7.4
- net J1_IN: now also F1.3, F1.4
- net J2_IN: now also F2.3, F2.4
- net J3_IN: now also F3.3, F3.4
- net J4_IN: now also F4.3, F4.4
