File: communications.kicad_sch (KiCad schematic)
At the start: 13 parts, among them CN1 PJ-3059-B, U41 DSLVDS1048PWR, U42 DSLVDS1047PWR

Commit message: Checkpoint
Connections:
- net DATA0 renamed HS_DATA0
- net DATA1 renamed HS_DATA1
- net DATA2 renamed HS_DATA2
- net DATA3 renamed HS_DATA3
Changed lines of the file:
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@@
 		)
 	)
-	(global_label "DATA1"
+	(global_label "HS_DATA1"
 		(shape input)
 		(at 167.64 116.84 0)
@@
 		)
 		(property "Intersheetrefs" "${INTERSHEET_REFS}"
-			(at 176.2495 116.84 0)
-			(effects
-				(font
-					(size 1.27 1.27)
-				)
-				(justify left)
-				(hide yes)
-			)
-		)
-	)
-	(global_label "DATA3"
+			(at 179.7571 116.84 0)
+			(effects
+				(font
+					(size 1.27 1.27)
+				)
+				(justify left)
+				(hide yes)
+			)
+		)
+	)
+	(global_label "HS_DATA3"
 		(shape input)
 		(at 167.64 121.92 0)
@@
 		)
 		(property "Intersheetrefs" "${INTERSHEET_REFS}"
-			(at 176.2495 121.92 0)
-			(effects
-				(font
-					(size 1.27 1.27)
-				)
-				(justify left)
-				(hide yes)
-			)
-		)
-	)
-	(global_label "DATA0"
+			(at 179.7571 121.92 0)
+			(effects
+				(font
+					(size 1.27 1.27)
+				)
+				(justify left)
+				(hide yes)
+			)
+		)
+	)
+	(global_label "HS_DATA0"
 		(shape input)
 		(at 167.64 114.3 0)
@@
 		)
 		(property "Intersheetrefs" "${INTERSHEET_REFS}"
-			(at 176.2495 114.3 0)
-			(effects
-				(font
-					(size 1.27 1.27)
-				)
-				(justify left)
-				(hide yes)
-			)
-		)
-	)
-	(global_label "DATA1"
+			(at 179.7571 114.3 0)
+			(effects
+				(font
+					(size 1.27 1.27)
+				)
+				(justify left)
+				(hide yes)
+			)
+		)
+	)
+	(global_label "HS_DATA1"
 		(shape input)
 		(at 167.64 67.31 0)
@@
 		)
 		(property "Intersheetrefs" "${INTERSHEET_REFS}"
-			(at 176.2495 67.31 0)
+			(at 179.7571 67.31 0)
 			(effects
 				(font
@@
 		)
 	)
-	(global_label "DATA2"
+	(global_label "HS_DATA2"
 		(shape input)
 		(at 167.64 69.85 0)
@@
 		)
 		(property "Intersheetrefs" "${INTERSHEET_REFS}"
-			(at 176.2495 69.85 0)
+			(at 179.7571 69.85 0)
 			(effects
 				(font
@@
 		)
 	)
-	(global_label "DATA3"
+	(global_label "HS_DATA3"
 		(shape input)
 		(at 167.64 72.39 0)
@@
 		)
 		(property "Intersheetrefs" "${INTERSHEET_REFS}"
-			(at 176.2495 72.39 0)
-			(effects
-				(font
-					(size 1.27 1.27)
-				)
-				(justify left)
-				(hide yes)
-			)
-		)
-	)
-	(global_label "DATA2"
+			(at 179.7571 72.39 0)
+			(effects
+				(font
+					(size 1.27 1.27)
+				)
+				(justify left)
+				(hide yes)
+			)
+		)
+	)
+	(global_label "HS_DATA2"
 		(shape input)
 		(at 167.64 119.38 0)
@@
 		)
 		(property "Intersheetrefs" "${INTERSHEET_REFS}"
-			(at 176.2495 119.38 0)
-			(effects
-				(font
-					(size 1.27 1.27)
-				)
-				(justify left)
-				(hide yes)
-			)
-		)
-	)
-	(global_label "DATA0"
+			(at 179.7571 119.38 0)
+			(effects
+				(font
+					(size 1.27 1.27)
+				)
+				(justify left)
+				(hide yes)
+			)
+		)
+	)
+	(global_label "HS_DATA0"
 		(shape input)
 		(at 167.64 64.77 0)
@@
 		)
 		(property "Intersheetrefs" "${INTERSHEET_REFS}"
-			(at 176.2495 64.77 0)
-			(effects
-				(font
+			(at 179.7571 64.77 0)
+			(effects
+				(font

Commit message: Checkpoint
Connections:
- net DOUT1-: now reaches RJ2.1, U42.16 (DOUT1-)
- net DOUT1+: now reaches RJ2.2, U42.15 (DOUT1+)
- net DOUT2+: now reaches RJ2.3, U42.14 (DOUT2+)
- net DOUT2-: now reaches RJ2.4, U42.13 (DOUT2-)
- net DOUT3-: now reaches RJ2.5, U42.12 (DOUT3-)
- net DOUT3+: now reaches RJ2.6, U42.11 (DOUT3+)
- net DOUT4+: now reaches RJ2.7, U42.10 (DOUT4+)
- net DOUT4-: now reaches RJ2.8, U42.9 (DOUT4-)
- net RIN1-: now reaches R20.1, RJ1.8, U41.1 (RIN1-)
- net RIN1+: now reaches R20.2, RJ1.7, U41.2 (RIN1+)
- net RIN2+: now reaches R21.1, RJ1.6, U41.3 (RIN2+)
- net RIN2-: now reaches R21.2, RJ1.5, U41.4 (RIN2-)
- net RIN4+: now reaches R23.1, RJ1.2, U41.7 (RIN4+)
- net RIN4-: now reaches R23.2, RJ1.1, U41.8 (RIN4-)
- net RIN3-: now reaches R22.1, RJ1.4, U41.5 (RIN3-)
- net RIN3+: now reaches R22.2, RJ1.3, U41.6 (RIN3+)

Commit message: Close to final, lots of cleanup, added back audio
Parts:
- removed CN1: PJ-3059-B, EasyEDA:AUDIO-TH_XKB_PJ-3059-B, symbol EasyEDA:PJ-3059-B
Other:
- note removed: "IR Control"

Commit message: Library shuffle and Fabrication Toolkit micro adjustments
Parts:
- C38, C40: footprint PCM_JLCPCB:C_0402 -> PixelBlit:C_0402; symbol PCM_JLCPCB-Capacitors:0402,100nF -> PixelBlit:0402,100nF
- C39, C41: footprint PCM_JLCPCB:C_0402 -> PixelBlit:C_0402; symbol PCM_JLCPCB-Capacitors:0402,1nF -> PixelBlit:0402,1nF
- R20, R21, R22, R23: footprint PCM_JLCPCB:R_0402 -> PixelBlit:R_0402; symbol PCM_JLCPCB-Resistors:0402,100Ω -> PixelBlit:0402,100Ω
- RJ1, RJ2: footprint EasyEDA:RJ45-TH_R-RJ45R08P-A004 -> PixelBlit:RJ45-TH_R-RJ45R08P-A004; symbol EasyEDA:R-RJ45R08P-A004 -> PixelBlit:R-RJ45R08P-A004
- U41: footprint EasyEDA:TSSOP-16_L5.0-W4.4-P0.65-LS6.4-BL -> PixelBlit:TSSOP-16_L5.0-W4.4-P0.65-LS6.4-BL; symbol EasyEDA:DSLVDS1048PWR -> PixelBlit:DSLVDS1048PWR
- U42: footprint EasyEDA:TSSOP-16_L5.0-W4.4-P0.65-LS6.4-TL -> PixelBlit:TSSOP-16_L5.0-W4.4-P0.65-LS6.4-TL; symbol EasyEDA:DSLVDS1047PWR -> PixelBlit:DSLVDS1047PWR
Changed lines of the file:
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@@
 	)
 	(symbol
-		(lib_id "EasyEDA:R-RJ45R08P-A004")
+		(lib_id "PixelBlit:R-RJ45R08P-A004")
 		(at 69.85 114.3 90)
 		(unit 1)
@@
 			)
 		)
-		(property "Footprint" "EasyEDA:RJ45-TH_R-RJ45R08P-A004"
+		(property "Footprint" "PixelBlit:RJ45-TH_R-RJ45R08P-A004"
 			(at 90.17 114.3 0)
 			(effects
@@
 	)
 	(symbol
-		(lib_id "power:+3V3")
+		(lib_id "PixelBlit:+3V3")
 		(at 154.94 92.71 0)
 		(unit 1)
@@
 	)
 	(symbol
-		(lib_id "PCM_JLCPCB-Resistors:0402,100Ω")
+		(lib_id "PixelBlit:0402,100Ω")
 		(at 138.43 58.42 0)
 		(unit 1)
@@
 			)
 		)
-		(property "Footprint" "PCM_JLCPCB:R_0402"
+		(property "Footprint" "PixelBlit:R_0402"
 			(at 136.652 58.42 90)
 			(effects
@@
 	)
 	(symbol
-		(lib_id "PCM_JLCPCB-Capacitors:0402,1nF")
+		(lib_id "PixelBlit:0402,1nF")
 		(at 162.56 96.52 0)
 		(unit 1)
@@
 			)
 		)
-		(property "Footprint" "PCM_JLCPCB:C_0402"
+		(property "Footprint" "PixelBlit:C_0402"
 			(at 160.782 96.52 90)
 			(effects
@@
 	)
 	(symbol
-		(lib_id "power:GND")
+		(lib_id "PixelBlit:GND")
 		(at 154.94 82.55 0)
 		(unit 1)
@@
 	)
 	(symbol
-		(lib_id "PCM_JLCPCB-Capacitors:0402,100nF")
+		(lib_id "PixelBlit:0402,100nF")
 		(at 157.48 96.52 0)
 		(unit 1)
@@
 			)
 		)
-		(property "Footprint" "PCM_JLCPCB:C_0402"
+		(property "Footprint" "PixelBlit:C_0402"
 			(at 155.702 96.52 90)
 			(effects
@@
 	)
 	(symbol
-		(lib_id "PCM_JLCPCB-Capacitors:0402,1nF")
+		(lib_id "PixelBlit:0402,1nF")
 		(at 162.56 49.53 0)
 		(unit 1)
@@
 			)
 		)
-		(property "Footprint" "PCM_JLCPCB:C_0402"
+		(property "Footprint" "PixelBlit:C_0402"
 			(at 160.782 49.53 90)
 			(effects
@@
 	)
 	(symbol
-		(lib_id "PCM_JLCPCB-Resistors:0402,100Ω")
+		(lib_id "PixelBlit:0402,100Ω")
 		(at 129.54 63.5 0)
 		(unit 1)
@@
 			)
 		)
-		(property "Footprint" "PCM_JLCPCB:R_0402"
+		(property "Footprint" "PixelBlit:R_0402"
 			(at 127.762 63.5 90)
 			(effects
@@
 	)
 	(symbol
-		(lib_id "power:+3V3")
+		(lib_id "PixelBlit:+3V3")
 		(at 154.94 45.72 0)
 		(unit 1)
@@
 	)
 	(symbol
-		(lib_id "PCM_JLCPCB-Capacitors:0402,100nF")
+		(lib_id "PixelBlit:0402,100nF")
 		(at 157.48 49.53 0)
 		(unit 1)
@@
 			)
 		)
-		(property "Footprint" "PCM_JLCPCB:C_0402"
+		(property "Footprint" "PixelBlit:C_0402"
 			(at 155.702 49.53 90)
 			(effects
@@
 	)
 	(symbol
-		(lib_id "PCM_JLCPCB-Resistors:0402,100Ω")
+		(lib_id "PixelBlit:0402,100Ω")
 		(at 111.76 73.66 0)
 		(unit 1)
@@
 			)
 		)
-		(property "Footprint" "PCM_JLCPCB:R_0402"
+		(property "Footprint" "PixelBlit:R_0402"
 			(at 109.982 73.66 90)
 			(effects
@@
 	)
 	(symbol
-		(lib_id "EasyEDA:DSLVDS1047PWR")
+		(lib_id "PixelBlit:DSLVDS1047PWR")
 		(at 154.94 116.84 180)
 		(unit 1)
@@
 			)
 		)
-		(property "Footprint" "EasyEDA:TSSOP-16_L5.0-W4.4-P0.65-LS6.4-TL"
+		(property "Footprint" "PixelBlit:TSSOP-16_L5.0-W4.4-P0.65-LS6.4-TL"
 			(at 154.94 100.33 0)
 			(effects
@@
 	)
 	(symbol
-		(lib_id "power:GND")
+		(lib_id "PixelBlit:GND")
 		(at 167.64 100.33 0)
 		(unit 1)
@@
 	)
 	(symbol
-		(lib_id "EasyEDA:DSLVDS1048PWR")
+		(lib_id "PixelBlit:DSLVDS1048PWR")
 		(at 154.94 68.58 0)
 		(unit 1)
@@
 			)
 		)
-		(property "Footprint" "EasyEDA:TSSOP-16_L5.0-W4.4-P0.65-LS6.4-BL"
+		(property "Footprint" "PixelBlit:TSSOP-16_L5.0-W4.4-P0.65-LS6.4-BL"
 			(at 154.94 85.09 0)
 			(effects
@@
 	)
 	(symbol
-		(lib_id "power:GND")
+		(lib_id "PixelBlit:GND")
 		(at 154.94 129.54 0)
 		(unit 1)
@@
 	)
 	(symbol
-		(lib_id "EasyEDA:R-RJ45R08P-A004")
+		(lib_id "PixelBlit:R-RJ45R08P-A004")
 		(at 69.85 62.23 90)
 		(unit 1)
@@
 			)
 		)
-		(property "Footprint" "EasyEDA:RJ45-TH_R-RJ45R08P-A004"
+		(property "Footprint" "PixelBlit:RJ45-TH_R-RJ45R08P-A004"
 			(at 90.17 62.23 0)
 			(effects
@@
 	)
 	(symbol
-		(lib_id "power:GND")
+		(lib_id "PixelBlit:GND")
 		(at 167.64 53.34 0)
 		(unit 1)
@@
 	)
 	(symbol
-		(lib_id "PCM_JLCPCB-Resistors:0402,100Ω")
+		(lib_id "PixelBlit:0402,100Ω")
 		(at 120.65 68.58 0)
 		(unit 1)
@@
 			)
 		)
-		(property "Footprint" "PCM_JLCPCB:R_0402"
+		(property "Footprint" "PixelBlit:R_0402"
 			(at 118.872 68.58 90)
 			(effects

Commit message: Fixes for second production run
Parts:
- removed U41: DSLVDS1048PWR, PixelBlit:TSSOP-16_L5.0-W4.4-P0.65-LS6.4-BL, symbol PixelBlit:DSLVDS1048PWR
- removed U42: DSLVDS1047PWR, PixelBlit:TSSOP-16_L5.0-W4.4-P0.65-LS6.4-TL, symbol PixelBlit:DSLVDS1047PWR
- added U41: DS90LV048ATMTCX_NOPB, JLCImport:DS90LV048ATMTCX_NOPB, symbol JLCImport:DS90LV048ATMTCX_NOPB
- added U42: DS90LV047ATMTCX_NOPB, JLCImport:DS90LV047ATMTCX_NOPB, symbol JLCImport:DS90LV047ATMTCX_NOPB
Connections:
- net +3V3: now also U41.13 (VCC), U42.1 (EN), U42.4 (VCC)
- net DATA_IN_EN: now also U41.16 (EN)
- net DOUT1+: now also U42.15 (DOUT1+)
- net DOUT1-: now also U42.16 (DOUT1-)
- net DOUT2+: now also U42.14 (DOUT2+)
- net DOUT2-: now also U42.13 (DOUT2-)
- net DOUT3+: now also U42.11 (DOUT3+)
- net DOUT3-: now also U42.12 (DOUT3-)
- net DOUT4+: now also U42.10 (DOUT4+)
- net DOUT4-: now also U42.9 (DOUT4-)
- net GND: now also U42.5 (GND)
- net HS_DATA0: now also U41.15 (ROUT1), U42.7 (DIN4)
- net HS_DATA1: now also U41.14 (ROUT2), U42.6 (DIN3)
- net HS_DATA2: now also U41.11 (ROUT3), U42.3 (DIN2)
- net HS_DATA3: now also U41.10 (ROUT4), U42.2 (DIN1)
- net RIN1+: now also U41.2 (RIN1+)
- net RIN1-: now also U41.1 (RIN1-)
- net RIN2+: now also U41.3 (RIN2+)
- net RIN2-: now also U41.4 (RIN2-)
- net RIN3+: now also U41.6 (RIN3+)
- net RIN3-: now also U41.5 (RIN3-)
- net RIN4+: now also U41.7 (RIN4+)
- net RIN4-: now also U41.8 (RIN4-)
- no-connect marks 1 -> 2
Changed lines of the file:
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@@
 	)
 	(junction
+		(at 154.94 52.07)
+		(diameter 0)
+		(color 0 0 0 0)
+	)
+	(junction
 		(at 129.54 67.31)
 		(diameter 0)
@@
 		(color 0 0 0 0)
 	)
-	(junction
-		(at 170.18 106.68)
-		(diameter 0)
-		(color 0 0 0 0)
+	(no_connect
+		(at 167.64 109.22)
 	)
 	(no_connect
@@
 	(wire
 		(pts
-			(xy 170.18 106.68) (xy 170.18 109.22)
-		)
-		(stroke
-			(width 0)
-			(type default)
-		)
-	)
-	(wire
-		(pts
 			(xy 82.55 64.77) (xy 120.65 64.77)
 		)
@@
 	(wire
 		(pts
-			(xy 154.94 45.72) (xy 154.94 54.61)
+			(xy 154.94 45.72) (xy 154.94 52.07)
 		)
 		(stroke
@@
 	(wire
 		(pts
-			(xy 170.18 109.22) (xy 167.64 109.22)
-		)
-		(stroke
-			(width 0)
-			(type default)
-		)
-	)
-	(wire
-		(pts
 			(xy 129.54 67.31) (xy 127 67.31)
 		)
@@
 	(wire
 		(pts
+			(xy 154.94 52.07) (xy 154.94 54.61)
+		)
+		(stroke
+			(width 0)
+			(type default)
+		)
+	)
+	(wire
+		(pts
 			(xy 109.22 77.47) (xy 109.22 72.39)
 		)
@@
 	)
 	(symbol
+		(lib_id "JLCImport:DS90LV047ATMTCX_NOPB")
+		(at 154.94 115.57 180)
+		(unit 1)
+		(exclude_from_sim no)
+		(in_bom yes)
+		(on_board yes)
+		(dnp no)
+		(property "Reference" "U42"
+			(at 147.32 99.06 0)
+			(effects
+				(font
+					(size 1.27 1.27)
+				)
+			)
+		)
+		(property "Value" "DS90LV047ATMTCX_NOPB"
+			(at 154.94 101.6 0)
+			(effects
+				(font
+					(size 1.27 1.27)
+				)
+			)
+		)
+		(property "Footprint" "JLCImport:DS90LV047ATMTCX_NOPB"
+			(at 154.94 115.57 0)
+			(effects
+				(font
+					(size 1.27 1.27)
+				)
+				(hide yes)
+			)
+		)
+		(property "Datasheet" "https://item.szlcsc.com/6534.html"
+			(at 154.94 115.57 0)
+			(effects
+				(font
+					(size 1.27 1.27)
+				)
+				(hide yes)
+			)
+		)
+		(property "Description" ""
+			(at 154.94 115.57 0)
+			(effects
+				(font
+					(size 1.27 1.27)
+				)
+				(hide yes)
+			)
+		)
+		(property "LCSC" "C87097"
+			(at 154.94 115.57 0)
+			(effects
+				(font
+					(size 1.27 1.27)
+				)
+				(hide yes)
+			)
+		)
+		(property "Manufacturer" "TI(德州仪器)"
+			(at 154.94 115.57 0)
+			(effects
+				(font
+					(size 1.27 1.27)
+				)
+				(hide yes)
+			)
+		)
+		(property "Manufacturer Part" "DS90LV047ATMTCX/NOPB"
+			(at 154.94 115.57 0)
+			(effects
+				(font
+					(size 1.27 1.27)
+				)
+				(hide yes)
+			)
+		)
+		(pin "15"
+		)
+		(pin "7"
+		)
+		(pin "10"
+		)
+		(pin "5"
+		)
+		(pin "6"
+		)
+		(pin "2"
+		)
+		(pin "4"
+		)
+		(pin "3"
+		)
+		(pin "9"
+		)
+		(pin "11"
+		)
+		(pin "16"
+		)
+		(pin "1"
+		)
+		(pin "13"
+		)
+		(pin "14"
+		)
+		(pin "8"
+		)
+		(pin "12"
+		)
+		(instances
+			(project ""
+				(path "/046bafbc-5afd-4d51-a157-fe6ddaf6697d/ba35bb49-3203-4382-af50-555a2d58b34d"
+					(reference "U42")
+					(unit 1)
+				)
+			)
+		)
+	)
+	(symbol
 		(lib_id "PixelBlit:GND")
 		(at 154.94 82.55 0)
@@
 	)
 	(symbol
-		(lib_id "PixelBlit:DSLVDS1047PWR")
-		(at 154.94 116.84 180)
+		(lib_name "DS90LV048ATMTCX_NOPB_1")
+		(lib_id "JLCImport:DS90LV048ATMTCX_NOPB")
+		(at 154.94 78.74 0)
 		(unit 1)
 		(exclude_from_sim no)
@@
 		(on_board yes)
 		(dnp no)
-		(property "Reference" "U42"
-			(at 144.272 99.568 0)
+		(fields_autoplaced yes)
+		(property "Reference" "U41"
+			(at 157.0833 52.07 0)
 			(effects
 				(font
 					(size 1.27 1.27)
 				)
-				(justify right)
+				(justify left)
 			)
 		)
-		(property "Value" "DSLVDS1047PWR"
-			(at 136.906 102.108 0)
+		(property "Value" "DS90LV048ATMTCX_NOPB"
+			(at 157.0833 54.61 0)
 			(effects
 				(font
 					(size 1.27 1.27)
 				)
-				(justify right)
+				(justify left)
 			)
 		)
-		(property "Footprint" "PixelBlit:TSSOP-16_L5.0-W4.4-P0.65-LS6.4-TL"
-			(at 154.94 100.33 0)
+		(property "Footprint" "JLCImport:DS90LV048ATMTCX_NOPB"
+			(at 154.94 78.74 0)
 			(effects
 				(font
@@
 			)
 		)
-		(property "Datasheet" ""
-			(at 154.94 116.84 0)
+		(property "Datasheet" "https://item.szlcsc.com/6534.html"
+			(at 154.94 78.74 0)
 			(effects
 				(font
@@
 		)
 		(property "Description" ""
-			(at 154.94 116.84 0)
+			(at 154.94 78.74 0)
 			(effects
 				(font
@@
 			)
 		)
-		(property "LCSC Part" "C2671205"
-			(at 154.94 97.79 0)
+		(property "LCSC" "C87137"
+			(at 154.94 78.74 0)
 			(effects
 				(font
@@
 			)
 		)
-		(pin "2"
+		(property "Manufacturer" "TI(德州仪器)"
+			(at 154.94 78.74 0)
+			(effects
+				(font
+					(size 1.27 1.27)
+				)
+				(hide yes)
+			)
 		)
-		(pin "1"
+		(property "Manufacturer Part" "DS90LV048ATMTCX/NOPB"
+			(at 154.94 78.74 0)
+			(effects
+				(font
+					(size 1.27 1.27)
+				)
+				(hide yes)
+			)
 		)
-		(pin "6"
+		(pin "5"
 		)
 		(pin "7"
@@
 		(pin "16"
 		)
-		(pin "15"
+		(pin "1"
 		)
-		(pin "14"
+		(pin "6"
+		)
+		(pin "9"
 		)
 		(pin "13"
 		)
-		(pin "12"
+		(pin "15"
+		)
+		(pin "14"
 		)
 		(pin "11"
@@
 		(pin "10"
 		)
-		(pin "9"
+		(pin "12"
 		)
-		(pin "4"
+		(pin "2"
 		)
-		(pin "5"
+		(pin "4"
 		)
 		(pin "3"
@@
 			(project ""
 				(path "/046bafbc-5afd-4d51-a157-fe6ddaf6697d/ba35bb49-3203-4382-af50-555a2d58b34d"
-					(reference "U42")
+					(reference "U41")
 					(unit 1)
 				)
@@
 					(unit 1)
 				)
-			)
-		)
-	)
-	(symbol
-		(lib_id "PixelBlit:DSLVDS1048PWR")
-		(at 154.94 68.58 0)
-		(unit 1)
-		(exclude_from_sim no)
-		(in_bom yes)
-		(on_board yes)
-		(dnp no)
-		(property "Reference" "U41"
-			(at 145.796 49.022 0)
-			(effects
-				(font
-					(size 1.27 1.27)
-				)
-				(justify left)
-			)
-		)
-		(property "Value" "DSLVDS1048PWR"
-			(at 137.414 51.054 0)
-			(effects
-				(font
-					(size 1.27 1.27)
-				)
-				(justify left)
-			)
-		)
-		(property "Footprint" "PixelBlit:TSSOP-16_L5.0-W4.4-P0.65-LS6.4-BL"
-			(at 154.94 85.09 0)
-			(effects
-				(font
-					(size 1.27 1.27)
-				)
-				(hide yes)
-			)
-		)
-		(property "Datasheet" ""
-			(at 154.94 68.58 0)
-			(effects
-				(font
-					(size 1.27 1.27)
-				)
-				(hide yes)
-			)
-		)
-		(property "Description" ""
-			(at 154.94 68.58 0)
-			(effects
-				(font
-					(size 1.27 1.27)
-				)
-				(hide yes)
-			)
-		)
-		(property "LCSC Part" "C2671655"
-			(at 154.94 87.63 0)
-			(effects
-				(font
-					(size 1.27 1.27)
-				)
-				(hide yes)
-			)
-		)
-		(pin "6"
-		)
-		(pin "5"
-		)
-		(pin "2"
-		)
-		(pin "1"
-		)
-		(pin "4"
-		)
-		(pin "7"
-		)
-		(pin "8"
-		)
-		(pin "16"
-		)
-		(pin "15"
-		)
-		(pin "14"
-		)
-		(pin "13"
-		)
-		(pin "12"
-		)
-		(pin "11"
-		)
-		(pin "10"
-		)
-		(pin "9"
-		)
-		(pin "3"
-		)
-		(instances
-			(project ""
-				(path "/046bafbc-5afd-4d51-a157-fe6ddaf6697d/ba35bb49-3203-4382-af50-555a2d58b34d"
-					(reference "U41")
-					(unit 1)
-				)
